File: Codeshelf-0008/Codeshelf-0008.v01.sch (EAGLE design)
At the start: 41 parts, among them IC1 74AHC1G04DCK, IC2 74AHC1G04DCK, IC3 74AHC1G04DCK, IC4 74AHC1G08DCK, IC5 74AHC1G08DCK, IC6 74AHC1G08DCK, J1 M05X2PTH, J2 POWER_JACKPTH, J3 M08X2, J4 M08X2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

Commit message: Changes reviewed with Charlie
Parts:
- removed LOGO: CODESHELF-LOGO, GW-devices:CODESHELF-LOGO
Changed lines of the file:
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@@
 <part name="+3V6" library="supply1" deviceset="+3V3" device=""/>
 <part name="+3V7" library="supply1" deviceset="+3V3" device=""/>
-<part name="LOGO" library="GW-devices" deviceset="CODESHELF-LOGO" device=""/>
 <part name="C5" library="GW-devices" deviceset="RF-C" device="0402" value=".1uF">
 <attribute name="MFGN" value="Murata"/>
@@
 <instance part="+3V6" gate="G$1" x="-71.12" y="86.36"/>
 <instance part="+3V7" gate="G$1" x="-180.34" y="45.72"/>
-<instance part="LOGO" gate="G$1" x="55.88" y="-124.46"/>
 <instance part="C5" gate="G$1" x="48.26" y="30.48" rot="R90">
 <attribute name="MFGN" x="48.26" y="30.48" size="1.778" layer="96" rot="R90" display="off"/>

Commit message: BOM review before first articles of 0005, 0007, 0008, 0012
Reviewed BOM with Charlie
Parts:
- D1, D2, R2, R3: NOTES (none) -> DNP
Changed lines of the file:
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@@
 <attribute name="MFGN" value="OSRAM"/>
 <attribute name="MFGP" value="Q62702P5182"/>
+<attribute name="NOTES" value="DNP"/>
 </part>
 <part name="D2" library="led" deviceset="LED" device="CHIP-LED0805" value="GREEN">
 <attribute name="MFGN" value="OSRAM"/>
 <attribute name="MFGP" value="Q65110P5179"/>
+<attribute name="NOTES" value="DNP"/>
 </part>
 <part name="R2" library="GW-devices" deviceset="RF-R" device="0402" value="220">
 <attribute name="MFGN" value="Panasonic"/>
 <attribute name="MFGP" value="ERJ-2GEJ224X"/>
+<attribute name="NOTES" value="DNP"/>
 </part>
 <part name="R3" library="GW-devices" deviceset="RF-R" device="0402" value="390">
 <attribute name="MFGN" value="Panasonic"/>
 <attribute name="MFGP" value="ERJ-2GEJ394X"/>
+<attribute name="NOTES" value="DNP"/>
 </part>
 <part name="C3" library="GW-devices" deviceset="RF-C" device="0603" value="100pF">
@@
 <part name="JF1" library="GW-devices" deviceset="JUMPER-2X" device="-SMT-VIA"/>
 <part name="JF2" library="GW-devices" deviceset="JUMPER-2X" device="-SMT-VIA"/>
+<part name="+3V8" library="supply1" deviceset="+3V3" device=""/>
 </parts>
 <sheets>
@@
 <attribute name="MFGN" x="-152.4" y="83.82" size="1.778" layer="96" rot="R270" display="off"/>
 <attribute name="MFGP" x="-152.4" y="83.82" size="1.778" layer="96" rot="R270" display="off"/>
+<attribute name="NOTES" x="-152.4" y="83.82" size="1.778" layer="96" rot="R270" display="off"/>
 </instance>
 <instance part="D2" gate="G$1" x="-152.4" y="76.2" rot="R270">
 <attribute name="MFGN" x="-152.4" y="76.2" size="1.778" layer="96" rot="R270" display="off"/>
 <attribute name="MFGP" x="-152.4" y="76.2" size="1.778" layer="96" rot="R270" display="off"/>
+<attribute name="NOTES" x="-152.4" y="76.2" size="1.778" layer="96" rot="R270" display="off"/>
 </instance>
 <instance part="R2" gate="G$1" x="-167.64" y="83.82">
 <attribute name="MFGN" x="-167.64" y="83.82" size="1.778" layer="96" display="off"/>
 <attribute name="MFGP" x="-167.64" y="83.82" size="1.778" layer="96" display="off"/>
+<attribute name="NOTES" x="-167.64" y="83.82" size="1.778" layer="96" display="off"/>
 </instance>
 <instance part="R3" gate="G$1" x="-167.64" y="76.2">
 <attribute name="MFGN" x="-167.64" y="76.2" size="1.778" layer="96" display="off"/>
 <attribute name="MFGP" x="-167.64" y="76.2" size="1.778" layer="96" display="off"/>
+<attribute name="NOTES" x="-167.64" y="76.2" size="1.778" layer="96" display="off"/>
 </instance>
 <instance part="C3" gate="G$1" x="-165.1" y="-5.08" rot="R90">
@@
 <instance part="JF1" gate="G$1" x="-167.64" y="35.56"/>
 <instance part="JF2" gate="G$1" x="-167.64" y="20.32"/>
+<instance part="+3V8" gate="G$1" x="-30.48" y="93.98"/>
 </instances>
 <busses>
@@
 </segment>
 <segment>
-<wire x1="-30.48" y1="86.36" x2="-30.48" y2="83.82" width="0.1524" layer="91"/>
+<wire x1="-30.48" y1="91.44" x2="-30.48" y2="83.82" width="0.1524" layer="91"/>
 <pinref part="R1" gate="G$1" pin="2"/>
 </segment>
