File: Codeshelf-0008/Codeshelf-0008.v01.sch.org.sch (EAGLE design)
At the start: 42 parts, among them IC1 74AHC1G04DCK, IC2 74AHC1G04DCK, IC4 74AHC1G08DCK, IC5 74AHC1G08DCK, IC6 74AHC1G08DCK, J1 M05X2PTH, J2 POWER_JACKPTH, J3 M08X2, J4 M08X2, Q1 MOSFET-NCHANNELBSS138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

Commit message: New position controller design
Parts:
- removed Q1, Q2: MOSFET-NCHANNELBSS138, SparkFun-DiscreteSemi:MOSFET-NCHANNELBSS138
- removed R4, R5, R6, R7: 10K, GW-devices:RF-R0402
- removed U$2, U$3, U$4: FIDUCIAL, adafruit:FIDUCIAL
- added C5, C6, C7, C8, C9: .1uF, GW-devices:RF-C0402
- added IC3: 74AHC1G04DCK, 74xx-little-us:74AHC1G04DCK
- added U2: MAX232SOIC16, SparkFun:MAX232SOIC16
- J1: NOTES DNP - flashing header -> (none)
- J3, J4: NOTES DNP - optional channels -> (none)
- JF1, JF2: NOTES DNP - flashing jumper -> (none)
- U6, U7, U8: value D-FLIP-FLOP-74LV1G79DBVR -> D-FLIP-FLOP-74LV1G79; device GW-devices:D-FLIP-FLOP-74LV1G79DBVR -> GW-devices:D-FLIP-FLOP-74LV1G79
Connections:
- new net C1: C5.1, U2.C1+
- new net C2: C6.1, U2.C2+
- new net N$11: C6.2, U2.C2-
- new net N$12: C7.1, U2.V-
- new net N$15: C8.1, U2.V+
- new net N$32: IC3A.O, U5.MR
- new net N$8: C5.2, U2.C1-
- net +3V3: now also C9.1, U2.VCC; no longer Q1.G, Q2.G, R4.1, R6.1
- net +5V: no longer R5.1, R7.1
- net GND: now also C7.2, C8.2, C9.2, U2.GND
- net N$1: now also U1.57; no longer U1.KBI0
- net N$2: now also U1.56; no longer U1.KBI1
- net N$25: now also IC3A.I; no longer U5.MR
- net SSI-CLK-3V3: no longer Q2.S, R6.2
- net SSI-CLK-5V: now also U2.T2OUT; no longer Q2.D, R7.2
- net SSI-TX-3V3: now also U2.T1IN; no longer Q1.S, R4.2
- net SSI-TX-5V: now also U2.T1OUT; no longer Q1.D, R5.2
