File: Codeshelf-0012/Codeshelf-0012.v01.brd (EAGLE design)
At the start: 56.6 x 57.7 mm, 24 parts, among them U1 ZSFM201-1A, U2 FT232RL, X1 USBPTH

Commit message: Changes reviewed with Charlie
Parts:
- removed U$2: CODESHELF-LOGO, GW-devices:CODESHELF-LOGO
- added U$1: (no value), GW-devices:CODESHELF-LOGO
Other:
- board text added: "CS0012.2013.11.24.n1"
- board text removed: "CS0012.v01.r01"
- board text removed: "Copyright 2013 Codeshelf, Inc"
Changed lines of the file:
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@@
 <wire x1="6.62" y1="32.85" x2="0" y2="32.85" width="0" layer="20"/>
 <wire x1="0" y1="32.85" x2="0" y2="0" width="0" layer="20"/>
-<text x="54.8" y="1.8" size="1.016" layer="25" rot="R90">Copyright 2013 Codeshelf, Inc</text>
-<text x="52.8" y="1.7" size="1.016" layer="25" rot="R90">CS0012.v01.r01</text>
+<text x="53.8" y="2.3" size="1.778" layer="25" rot="R90">CS0012.2013.11.24.n1</text>
 <hole x="14.31" y="14.83" drill="3.2"/>
 <hole x="14.31" y="42.83" drill="3.2"/>
@@
 <attribute name="MFGP" value="MICROSMD050F-2" x="4" y="43.5" size="1.778" layer="27" display="off"/>
 </element>
-<element name="U$2" library="GW-devices" package="CODESHELF-LOGO" value="CODESHELF-LOGO" x="46.7" y="27.1" rot="R90"/>
+<element name="U$1" library="GW-devices" package="CODESHELF-LOGO" value="" x="49.1" y="4.2" rot="R90"/>
 </elements>
 <signals>
