File: Codeshelf-0012/Codeshelf-0012.v01.sch (EAGLE design)
At the start: 24 parts, among them U1 ZSFM201-1A, U2 FT232RL, X1 USBPTH

Commit message: Changes related to design review with Ravi and Charlie.
Mainly we need a new way to connect all of the boards where the cables
enter the back.
Parts:
- R1: MFGN (none) -> Pansonic; MFGP (none) -> ERJ-2GEJ104X; PRICE (none) -> 0.10
Changed lines of the file:
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@@
 <attribute name="MFGP" value="GRM155R61A104KA01D"/>
 </part>
-<part name="R1" library="GW-devices" deviceset="RF-R" device="0402" value="100K"/>
+<part name="R1" library="GW-devices" deviceset="RF-R" device="0402" value="100K">
+<attribute name="MFGN" value="Pansonic"/>
+<attribute name="MFGP" value="ERJ-2GEJ104X"/>
+<attribute name="PRICE" value="0.10"/>
+</part>
 <part name="+3V4" library="supply1" deviceset="+3V3" device=""/>
 <part name="C6" library="GW-devices" deviceset="RF-C" device="0402" value="1nF">
@@
 <attribute name="MFGP" x="-96.52" y="43.18" size="1.778" layer="96" display="off"/>
 </instance>
-<instance part="R1" gate="G$1" x="40.64" y="27.94" rot="R90"/>
+<instance part="R1" gate="G$1" x="40.64" y="27.94" rot="R90">
+<attribute name="MFGN" x="40.64" y="27.94" size="1.778" layer="96" rot="R90" display="off"/>
+<attribute name="MFGP" x="40.64" y="27.94" size="1.778" layer="96" rot="R90" display="off"/>
+<attribute name="PRICE" x="40.64" y="27.94" size="1.778" layer="96" rot="R90" display="off"/>
+</instance>
 <instance part="+3V4" gate="G$1" x="40.64" y="43.18"/>
 <instance part="C6" gate="G$1" x="40.64" y="10.16">

Commit message: Changes reviewed with Charlie
Parts:
- removed U$2: CODESHELF-LOGO, GW-devices:CODESHELF-LOGO
Changed lines of the file:
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@@
 <attribute name="MFGP" value="MICROSMD050F-2"/>
 </part>
-<part name="U$2" library="GW-devices" deviceset="CODESHELF-LOGO" device=""/>
 </parts>
 <sheets>
@@
 <attribute name="MFGP" x="-251.46" y="0" size="1.778" layer="96" rot="R90" display="off"/>
 </instance>
-<instance part="U$2" gate="G$1" x="-134.62" y="-53.34"/>
 </instances>
 <busses>

Commit message: BOM review before first articles of 0005, 0007, 0008, 0012
Reviewed BOM with Charlie
Parts:
- C6: MFGP GRM033R71C102KD01D -> GRM155R71C102KA01D
Changed lines of the file:
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@@
 <part name="C6" library="GW-devices" deviceset="RF-C" device="0402" value="1nF">
 <attribute name="MFGN" value="Murata"/>
-<attribute name="MFGP" value="GRM033R71C102KD01D"/>
+<attribute name="MFGP" value="GRM155R71C102KA01D"/>
 </part>
 <part name="GND4" library="supply1" deviceset="GND" device=""/>

Commit message: gitignore fixup
Parts:
- C1, C2: MFGP GRM1555C1H150JZ01 -> GJM1555C1H150JB01D
- C7: MFGP GRM219R61A475KE19D -> GRM219R61A475KE34J
Changed lines of the file:
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@@
 <part name="C1" library="GW-devices" deviceset="RF-C" device="0402" value="15pF">
 <attribute name="MFGN" value="Murata"/>
-<attribute name="MFGP" value="GRM1555C1H150JZ01"/>
+<attribute name="MFGP" value="GJM1555C1H150JB01D"/>
 </part>
 <part name="C2" library="GW-devices" deviceset="RF-C" device="0402" value="15pF">
 <attribute name="MFGN" value="Murata"/>
-<attribute name="MFGP" value="GRM1555C1H150JZ01"/>
+<attribute name="MFGP" value="GJM1555C1H150JB01D"/>
 </part>
 <part name="C3" library="GW-devices" deviceset="RF-C" device="0402" value="0.1µF">
@@
 <part name="C7" library="GW-devices" deviceset="RF-C" device="0805" value="4.7µF">
 <attribute name="MFGN" value="Murata"/>
-<attribute name="MFGP" value="GRM219R61A475KE19D"/>
+<attribute name="MFGP" value="GRM219R61A475KE34J"/>
 </part>
 <part name="C8" library="GW-devices" deviceset="RF-C" device="0402" value="0.1µF">
