File: Codeshelf-0007/Codeshelf-0007.v02.brd (EAGLE design)
At the start: 103.5 x 53 mm, 26 parts, among them J1 RJ45-8PTH, J2 RJ45-8PTH, U2 MC9S08QG-DT, U3 CAT9552, U4 RS485SOIC, U7 7SEGMENT-2DIGIT

Commit message: New position controller design
Parts:
- added U$1, U$2, U$3: FIDUCIAL, adafruit:FIDUCIAL_1MM
- moved J2 8.00 mm to (6.00, 26.5), turned to 90 degrees
- moved J1 7.60 mm to (97.0, 26.5), turned to 270 degrees
Routing:
- net +3V3: track 264.2 -> 242.7 mm
- net RS485_N: track 140.0 -> 138.0 mm
- net RS485_P: track 133.4 -> 134.7 mm
Other:
- board text added: "CS0007.2014.01.28.n1"
- board text removed: "CS0007.2013.11.24.n1"
