File: Codeshelf-0004/Codeshelf-0004.v02.brd (EAGLE design)
At the start: 13 parts, among them J5 HEADER-2X-2.54MM

Commit message: SlotFlex Pos. Controller, SMPS
Copied position controller elements to Slotflex schematic. Corrected
inductor value typo in SMPS.
Parts:
- L1: value 150uH -> 1.5uH
Changed lines of the file:
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@@
 <attribute name="PRICE" value="0.03" x="11.9" y="27.6" size="1.778" layer="27" rot="R270" display="off"/>
 </element>
-<element name="L1" library="GW-devices" package="SLF10165" value="150uH" x="15.5" y="35.2" smashed="yes" rot="R90">
+<element name="L1" library="GW-devices" package="SLF10165" value="1.5uH" x="15.5" y="35.2" smashed="yes" rot="R90">
 <attribute name="NAME" x="22.1" y="34.3" size="1.27" layer="25" rot="R90"/>
 <attribute name="MFGN" value="TDK" x="15.5" y="35.2" size="1.778" layer="27" rot="R90" display="off"/>

Commit message: Fixed FB resistor label
Made FB1/FB2 resistor label consistent with datasheet. but NOT with
online calculator
Parts:
- RFB1: value 45.3K -> 143K
- RFB2: value 143K -> 45.3K
- moved RFB1 3.67 mm to (10.0, 27.6)
- moved RFB2 3.67 mm to (11.6, 24.3)
Connections:
- net +3V3: now also RFB1.2; no longer RFB2.2
- net GND: now also RFB2.1; no longer RFB1.1
- net N$24: now also RFB1.1, RFB2.2; no longer RFB1.2, RFB2.1
Changed lines of the file:
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@@
 <attribute name="PRICE" value="1.23" x="15.5" y="35.2" size="1.778" layer="27" rot="R90" display="off"/>
 </element>
-<element name="RFB2" library="GW-devices" package="RF-R0402" value="143K" x="10" y="27.6" smashed="yes" rot="R90">
+<element name="RFB1" library="GW-devices" package="RF-R0402" value="143K" x="10" y="27.6" smashed="yes" rot="R90">
 <attribute name="NAME" x="8.87" y="26.11" size="1.27" layer="25" rot="R90"/>
 <attribute name="MFGN" value="Vishay" x="10" y="27.6" size="1.778" layer="27" rot="R90" display="off"/>
@@
 <attribute name="PRICE" value="0.05" x="10" y="27.6" size="1.778" layer="27" rot="R90" display="off"/>
 </element>
-<element name="RFB1" library="GW-devices" package="RF-R0402" value="45.3K" x="11.6" y="24.3" smashed="yes" rot="R90">
+<element name="RFB2" library="GW-devices" package="RF-R0402" value="45.3K" x="11.6" y="24.3" smashed="yes" rot="R90">
 <attribute name="NAME" x="12.3" y="18.75" size="1.27" layer="25" rot="R90"/>
 <attribute name="MFGN" value="Vishay" x="11.6" y="24.3" size="1.778" layer="27" rot="R90" display="off"/>
@@
 <contactref element="U-P1" pad="EXP"/>
 <contactref element="CSS" pad="2"/>
-<contactref element="RFB1" pad="1"/>
+<contactref element="RFB2" pad="1"/>
 <contactref element="COUT1" pad="2"/>
 <contactref element="REN2" pad="1"/>
@@
 <signal name="+3V3" class="1">
 <contactref element="L1" pad="2"/>
-<contactref element="RFB2" pad="2"/>
+<contactref element="RFB1" pad="2"/>
 <contactref element="CCOMP" pad="2"/>
 <contactref element="COUT1" pad="1"/>
@@
 <signal name="N$24">
 <contactref element="U-P1" pad="16"/>
-<contactref element="RFB2" pad="1"/>
-<contactref element="RFB1" pad="2"/>
+<contactref element="RFB1" pad="1"/>
+<contactref element="RFB2" pad="2"/>
 <contactref element="RCOMP" pad="2"/>
 <wire x1="11.6" y1="24.8" x2="13.2" y2="24.8" width="0.4064" layer="1"/>
