File: Codeshelf-0013/Codeshelf-0013.v00.sch (EAGLE design)
At the start: 28 parts, among them IC1 AT45DB161D8S1

Commit message: KW2 and Slotflex edits
Removed RTC crystal from KW2, fixed (connected) switches in schematic of
0009.v02 and Slotflex v3 with RJ45 with NEW pinout (compatible with new
scanner pinout which doesn't exist yet in a CHE).
Parts:
- removed C3, C4: 12pF, GW-devices:RF-C0402
- removed U$3: 32KHZ, KW2:32KHZ
Connections:
- removed net N$3: C4.1, U$1.XTAL32, U$3.1
- removed net N$4: C3.1, U$1.EXTAL32, U$3.2
- net GND: no longer C3.2, C4.2
Changed lines of the file:
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@@
 <part name="C1" library="GW-devices" deviceset="RF-C" device="0402" value="12pF"/>
 <part name="C2" library="GW-devices" deviceset="RF-C" device="0402" value="12pF"/>
-<part name="U$3" library="KW2" deviceset="32KHZ" device=""/>
-<part name="C3" library="GW-devices" deviceset="RF-C" device="0402" value="12pF"/>
-<part name="C4" library="GW-devices" deviceset="RF-C" device="0402" value="12pF"/>
-<part name="GND3" library="supply1" deviceset="GND" device=""/>
-<part name="GND4" library="supply1" deviceset="GND" device=""/>
 <part name="C5" library="GW-devices" deviceset="RF-C" device="0402" value="0.1uF"/>
 <part name="C6" library="GW-devices" deviceset="RF-C" device="0402" value="1000pF"/>
@@
 <instance part="C1" gate="G$1" x="-91.44" y="25.4"/>
 <instance part="C2" gate="G$1" x="-127" y="25.4" rot="R180"/>
-<instance part="U$3" gate="G$1" x="-116.84" y="53.34"/>
-<instance part="C3" gate="G$1" x="-104.14" y="50.8"/>
-<instance part="C4" gate="G$1" x="-132.08" y="50.8"/>
-<instance part="GND3" gate="1" x="-132.08" y="40.64"/>
-<instance part="GND4" gate="1" x="-104.14" y="40.64"/>
 <instance part="C5" gate="G$1" x="2.54" y="76.2" rot="R180"/>
 <instance part="C6" gate="G$1" x="-7.62" y="76.2" rot="R180"/>
@@
 </segment>
 <segment>
-<pinref part="GND3" gate="1" pin="GND"/>
-<pinref part="C4" gate="G$1" pin="2"/>
-<wire x1="-132.08" y1="43.18" x2="-132.08" y2="45.72" width="0.1524" layer="91"/>
-</segment>
-<segment>
-<pinref part="C3" gate="G$1" pin="2"/>
-<pinref part="GND4" gate="1" pin="GND"/>
-<wire x1="-104.14" y1="43.18" x2="-104.14" y2="45.72" width="0.1524" layer="91"/>
-</segment>
-<segment>
 <pinref part="C5" gate="G$1" pin="2"/>
 <pinref part="C6" gate="G$1" pin="2"/>
@@
 </segment>
 </net>
-<net name="N$3" class="0">
-<segment>
-<pinref part="U$3" gate="G$1" pin="1"/>
-<pinref part="C4" gate="G$1" pin="1"/>
-<wire x1="-121.92" y1="53.34" x2="-132.08" y2="53.34" width="0.1524" layer="91"/>
-<pinref part="U$1" gate="G$1" pin="XTAL32"/>
-<wire x1="-66.04" y1="35.56" x2="-66.04" y2="45.72" width="0.1524" layer="91"/>
-<wire x1="-66.04" y1="45.72" x2="-93.98" y2="45.72" width="0.1524" layer="91"/>
-<wire x1="-93.98" y1="45.72" x2="-93.98" y2="60.96" width="0.1524" layer="91"/>
-<wire x1="-93.98" y1="60.96" x2="-132.08" y2="60.96" width="0.1524" layer="91"/>
-<wire x1="-132.08" y1="60.96" x2="-132.08" y2="53.34" width="0.1524" layer="91"/>
-<junction x="-132.08" y="53.34"/>
-</segment>
-</net>
-<net name="N$4" class="0">
-<segment>
-<pinref part="U$3" gate="G$1" pin="2"/>
-<pinref part="C3" gate="G$1" pin="1"/>
-<wire x1="-111.76" y1="53.34" x2="-104.14" y2="53.34" width="0.1524" layer="91"/>
-<wire x1="-104.14" y1="53.34" x2="-96.52" y2="53.34" width="0.1524" layer="91"/>
-<junction x="-104.14" y="53.34"/>
-<pinref part="U$1" gate="G$1" pin="EXTAL32"/>
-<wire x1="-96.52" y1="53.34" x2="-96.52" y2="43.18" width="0.1524" layer="91"/>
-<wire x1="-96.52" y1="43.18" x2="-71.12" y2="43.18" width="0.1524" layer="91"/>
-<wire x1="-71.12" y1="43.18" x2="-71.12" y2="33.02" width="0.1524" layer="91"/>
-<wire x1="-71.12" y1="33.02" x2="-66.04" y2="33.02" width="0.1524" layer="91"/>
-</segment>
-</net>
