File: Codeshelf-0009/Codeshelf-0009.v03.sch (EAGLE design)
At the start: 21 parts, among them U1 MC9S08QG-DT, U3 RS485SOIC, U4 CAT9552

Commit message: Completed new PosCon
Added BOM (csv and excel) and prepared bottom silkscreen.
Parts:
- BDM, LED1, LED2, U$3, U$4: NOTES (none) -> DNP
- C1, C2: MFGP GRM033R61A104KE15D -> GRM155R61A104KA01D
- J1-PROG, J2: MFGN (none) -> Molex; MFGP (none) -> 0955016649; PRICE (none) -> 0.89
- SW-ACK: value SWITCH-TACTILE-320.03E11 -> SWITCH-TACTILE-320.01E11WHT; device GW-devices:SWITCH-TACTILE-320.03E11 -> GW-devices:SWITCH-TACTILE-320.01E11WHT; MFGP (none) -> 320.01E11WHT
- U$5: MFGN (none) -> Worldsemi; MFGP (none) -> WS2812
- U4: value CAT9552 -> PCA9552; device GW-devices:CAT9552 -> GW-devices:PCA9552
- renumbered U$1 to J1-PROG, U$2 to U$5, U$2-PROG to J2
Changed lines of the file:
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@@
 <part name="C1" library="GW-devices" deviceset="RF-C" device="0402" value=".1uF">
 <attribute name="MFGN" value="Murata"/>
-<attribute name="MFGP" value="GRM033R61A104KE15D"/>
+<attribute name="MFGP" value="GRM155R61A104KA01D"/>
 <attribute name="PRICE" value="0.02"/>
 </part>
@@
 <part name="+3V8" library="supply1" deviceset="+3V3" device=""/>
 <part name="GND8" library="supply1" deviceset="GND" device=""/>
-<part name="BDM" library="GW-devices" deviceset="TP2X4SMD" device=""/>
+<part name="BDM" library="GW-devices" deviceset="TP2X4SMD" device="">
+<attribute name="NOTES" value="DNP"/>
+</part>
 <part name="R1" library="GW-devices" deviceset="RF-R" device="0402" value="3.3K">
 <attribute name="MFGN" value="Panasonic"/>
@@
 <part name="C2" library="GW-devices" deviceset="RF-C" device="0402" value=".1uF">
 <attribute name="MFGN" value="Murata"/>
-<attribute name="MFGP" value="GRM033R61A104KE15D"/>
+<attribute name="MFGP" value="GRM155R61A104KA01D"/>
 <attribute name="PRICE" value="0.02"/>
 </part>
@@
 <attribute name="PRICE" value="4.29"/>
 </part>
-<part name="U4" library="GW-devices" deviceset="CAT9552" device=""/>
+<part name="U4" library="GW-devices" deviceset="PCA9552" device=""/>
 <part name="GND12" library="supply1" deviceset="GND" device=""/>
 <part name="GND13" library="supply1" deviceset="GND" device=""/>
@@
 </part>
 <part name="+3V5" library="supply1" deviceset="+3V3" device=""/>
-<part name="LED2" library="GW-devices" deviceset="7SEGMENT-1DIGIT" device="SMD"/>
-<part name="LED1" library="GW-devices" deviceset="7SEGMENT-1DIGIT" device="SMD"/>
+<part name="LED2" library="GW-devices" deviceset="7SEGMENT-1DIGIT" device="SMD">
+<attribute name="NOTES" value="DNP"/>
+</part>
+<part name="LED1" library="GW-devices" deviceset="7SEGMENT-1DIGIT" device="SMD">
+<attribute name="NOTES" value="DNP"/>
+</part>
 <part name="+3V3" library="supply1" deviceset="+3V3" device=""/>
 <part name="+3V6" library="supply1" deviceset="+3V3" device=""/>
 <part name="GND5" library="supply1" deviceset="GND" device=""/>
-<part name="SW-ACK" library="GW-devices" deviceset="SWITCH-TACTILE" device="-320.03E11"/>
-<part name="U$3" library="GW-devices" deviceset="SWITCH-TACTILE" device="" value="SWITCH-TACTILE"/>
-<part name="U$4" library="GW-devices" deviceset="SWITCH-TACTILE" device="" value="SWITCH-TACTILE"/>
-<part name="U$1" library="GW-devices" deviceset="RJ45-8" device=""/>
-<part name="U$2-PROG" library="GW-devices" deviceset="RJ45-8" device=""/>
-<part name="U$2" library="GW-devices" deviceset="WS2812" device=""/>
+<part name="SW-ACK" library="GW-devices" deviceset="SWITCH-TACTILE" device="-320.01E11WHT">
+<attribute name="MFGP" value="320.01E11WHT"/>
+</part>
+<part name="U$3" library="GW-devices" deviceset="SWITCH-TACTILE" device="" value="SWITCH-TACTILE">
+<attribute name="NOTES" value="DNP"/>
+</part>
+<part name="U$4" library="GW-devices" deviceset="SWITCH-TACTILE" device="" value="SWITCH-TACTILE">
+<attribute name="NOTES" value="DNP"/>
+</part>
+<part name="J1-PROG" library="GW-devices" deviceset="RJ45-8" device="">
+<attribute name="MFGN" value="Molex"/>
+<attribute name="MFGP" value="0955016649"/>
+<attribute name="PRICE" value="0.89"/>
+</part>
+<part name="J2" library="GW-devices" deviceset="RJ45-8" device="">
+<attribute name="MFGN" value="Molex"/>
+<attribute name="MFGP" value="0955016649"/>
+<attribute name="PRICE" value="0.89"/>
+</part>
+<part name="U$5" library="GW-devices" deviceset="WS2812" device="">
+<attribute name="MFGN" value="Worldsemi"/>
+<attribute name="MFGP" value="WS2812"/>
+</part>
 <part name="GND2" library="supply1" deviceset="GND" device=""/>
 <part name="+3V7" library="supply1" deviceset="+3V3" device=""/>
@@
 <instance part="BDM" gate="G$1" x="-63.5" y="30.48" smashed="yes" rot="MR0">
 <attribute name="NAME" x="-59.436" y="38.862" size="1.778" layer="95" rot="MR0"/>
+<attribute name="NOTES" x="-63.5" y="30.48" size="1.778" layer="96" rot="MR0" display="off"/>
 </instance>
 <instance part="R1" gate="G$1" x="-43.18" y="33.02">
@@
 </instance>
 <instance part="+3V5" gate="G$1" x="-73.66" y="81.28"/>
-<instance part="LED2" gate="G$1" x="-274.32" y="81.28"/>
-<instance part="LED1" gate="G$1" x="-243.84" y="81.28"/>
+<instance part="LED2" gate="G$1" x="-274.32" y="81.28">
+<attribute name="NOTES" x="-274.32" y="81.28" size="1.778" layer="96" display="off"/>
+</instance>
+<instance part="LED1" gate="G$1" x="-243.84" y="81.28">
+<attribute name="NOTES" x="-243.84" y="81.28" size="1.778" layer="96" display="off"/>
+</instance>
 <instance part="+3V3" gate="G$1" x="-307.34" y="109.22"/>
 <instance part="+3V6" gate="G$1" x="-307.34" y="60.96"/>
 <instance part="GND5" gate="1" x="144.78" y="7.62"/>
 <instance part="SW-ACK" gate="G$1" x="124.46" y="27.94"/>
-<instance part="U$3" gate="G$1" x="124.46" y="58.42"/>
-<instance part="U$4" gate="G$1" x="124.46" y="43.18"/>
-<instance part="U$1" gate="G$1" x="170.18" y="-20.32"/>
-<instance part="U$2-PROG" gate="G$1" x="170.18" y="-66.04"/>
-<instance part="U$2" gate="G$1" x="10.16" y="-66.04"/>
+<instance part="U$3" gate="G$1" x="124.46" y="58.42">
+<attribute name="NOTES" x="124.46" y="58.42" size="1.778" layer="96" display="off"/>
+</instance>
+<instance part="U$4" gate="G$1" x="124.46" y="43.18">
+<attribute name="NOTES" x="124.46" y="43.18" size="1.778" layer="96" display="off"/>
+</instance>
+<instance part="J1-PROG" gate="G$1" x="170.18" y="-20.32">
+<attribute name="MFGN" x="170.18" y="-20.32" size="1.778" layer="96" display="off"/>
+<attribute name="MFGP" x="170.18" y="-20.32" size="1.778" layer="96" display="off"/>
+<attribute name="PRICE" x="170.18" y="-20.32" size="1.778" layer="96" display="off"/>
+</instance>
+<instance part="J2" gate="G$1" x="170.18" y="-66.04">
+<attribute name="MFGN" x="170.18" y="-66.04" size="1.778" layer="96" display="off"/>
+<attribute name="MFGP" x="170.18" y="-66.04" size="1.778" layer="96" display="off"/>
+<attribute name="PRICE" x="170.18" y="-66.04" size="1.778" layer="96" display="off"/>
+</instance>
+<instance part="U$5" gate="G$1" x="10.16" y="-66.04">
+<attribute name="MFGN" x="10.16" y="-66.04" size="1.778" layer="96" display="off"/>
+<attribute name="MFGP" x="10.16" y="-66.04" size="1.778" layer="96" display="off"/>
+</instance>
 <instance part="GND2" gate="1" x="-7.62" y="-81.28"/>
 <instance part="+3V7" gate="G$1" x="7.62" y="-43.18"/>
@@
 <junction x="137.16" y="-58.42"/>
 <wire x1="137.16" y1="-71.12" x2="157.48" y2="-71.12" width="0.1524" layer="91"/>
-<pinref part="U$1" gate="G$1" pin="2"/>
-<pinref part="U$1" gate="G$1" pin="7"/>
-<pinref part="U$2-PROG" gate="G$1" pin="2"/>
-<pinref part="U$2-PROG" gate="G$1" pin="7"/>
+<pinref part="J1-PROG" gate="G$1" pin="2"/>
+<pinref part="J1-PROG" gate="G$1" pin="7"/>
+<pinref part="J2" gate="G$1" pin="2"/>
+<pinref part="J2" gate="G$1" pin="7"/>
 </segment>
 <segment>
@@
 </segment>
 <segment>
-<pinref part="U$2" gate="G$1" pin="GND"/>
+<pinref part="U$5" gate="G$1" pin="GND"/>
 <pinref part="GND2" gate="1" pin="GND"/>
 <wire x1="-5.08" y1="-71.12" x2="-7.62" y2="-71.12" width="0.1524" layer="91"/>
@@
 <junction x="139.7" y="-55.88"/>
 <wire x1="157.48" y1="-73.66" x2="139.7" y2="-73.66" width="0.1524" layer="91"/>
-<pinref part="U$1" gate="G$1" pin="1"/>
-<pinref part="U$1" gate="G$1" pin="8"/>
-<pinref part="U$2-PROG" gate="G$1" pin="1"/>
-<pinref part="U$2-PROG" gate="G$1" pin="8"/>
+<pinref part="J1-PROG" gate="G$1" pin="1"/>
+<pinref part="J1-PROG" gate="G$1" pin="8"/>
+<pinref part="J2" gate="G$1" pin="1"/>
+<pinref part="J2" gate="G$1" pin="8"/>
 </segment>
 <segment>
@@
 </segment>
 <segment>
-<pinref part="U$2" gate="G$1" pin="VDD"/>
+<pinref part="U$5" gate="G$1" pin="VDD"/>
 <wire x1="-5.08" y1="-66.04" x2="-10.16" y2="-66.04" width="0.1524" layer="91"/>
 <wire x1="-10.16" y1="-66.04" x2="-10.16" y2="-48.26" width="0.1524" layer="91"/>
@@
 <wire x1="7.62" y1="-48.26" x2="25.4" y2="-48.26" width="0.1524" layer="91"/>
 <wire x1="25.4" y1="-48.26" x2="25.4" y2="-60.96" width="0.1524" layer="91"/>
-<pinref part="U$2" gate="G$1" pin="VCC"/>
+<pinref part="U$5" gate="G$1" pin="VCC"/>
 <wire x1="25.4" y1="-60.96" x2="22.86" y2="-60.96" width="0.1524" layer="91"/>
 <pinref part="+3V7" gate="G$1" pin="+3V3"/>
@@
 <junction x="114.3" y="-33.02"/>
 <wire x1="157.48" y1="-17.78" x2="114.3" y2="-17.78" width="0.1524" layer="91"/>
-<pinref part="U$1" gate="G$1" pin="4"/>
-<pinref part="U$2-PROG" gate="G$1" pin="4"/>
+<pinref part="J1-PROG" gate="G$1" pin="4"/>
+<pinref part="J2" gate="G$1" pin="4"/>
 </segment>
 </net>
@@
 <wire x1="-50.8" y1="50.8" x2="104.14" y2="50.8" width="0.1524" layer="91"/>
 <wire x1="104.14" y1="50.8" x2="104.14" y2="-22.86" width="0.1524" layer="91"/>
-<pinref part="U$1" gate="G$1" pin="6"/>
+<pinref part="J1-PROG" gate="G$1" pin="6"/>
 <wire x1="157.48" y1="-22.86" x2="104.14" y2="-22.86" width="0.1524" layer="91"/>
 </segment>
@@
 <wire x1="-73.66" y1="58.42" x2="109.22" y2="58.42" width="0.1524" layer="91"/>
 <wire x1="109.22" y1="58.42" x2="109.22" y2="-15.24" width="0.1524" layer="91"/>
-<pinref part="U$1" gate="G$1" pin="3"/>
+<pinref part="J1-PROG" gate="G$1" pin="3"/>
 <wire x1="157.48" y1="-15.24" x2="109.22" y2="-15.24" width="0.1524" layer="91"/>
 </segment>
@@
 <wire x1="121.92" y1="-66.04" x2="157.48" y2="-66.04" width="0.1524" layer="91"/>
 <wire x1="121.92" y1="-20.32" x2="157.48" y2="-20.32" width="0.1524" layer="91"/>
-<pinref part="U$1" gate="G$1" pin="5"/>
-<pinref part="U$2-PROG" gate="G$1" pin="5"/>
+<pinref part="J1-PROG" gate="G$1" pin="5"/>
+<pinref part="J2" gate="G$1" pin="5"/>
 </segment>
 </net>
@@
 <net name="N$3" class="0">
 <segment>
-<pinref part="U$2" gate="G$1" pin="DI"/>
+<pinref part="U$5" gate="G$1" pin="DI"/>
 <wire x1="22.86" y1="-66.04" x2="30.48" y2="-66.04" width="0.1524" layer="91"/>
 <wire x1="30.48" y1="-66.04" x2="30.48" y2="-33.02" width="0.1524" layer="91"/>
