File: POSCON.PCB/POSCON.PCB.sch (EAGLE design)
At the start: 21 parts, among them J1-PROG RJ45-8, J2 RJ45-8, U1 MC9S08QG-DT, U3 RS485SOIC, U4 PCA9552

Commit message: Fixed BOM
Fixed PCA9552 P/N, Eswitch price, RGB LED DNP and BOM format.
Parts:
- SW-ACK: PRICE (none) -> 1.38
- U$5: NOTES (none) -> DNP
- U4: MFGP (none) -> PCA9552PW,112
Changed lines of the file:
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@@
 <attribute name="PRICE" value="4.29"/>
 </part>
-<part name="U4" library="GW-devices" deviceset="PCA9552" device=""/>
+<part name="U4" library="GW-devices" deviceset="PCA9552" device="">
+<attribute name="MFGP" value="PCA9552PW,112"/>
+</part>
 <part name="GND12" library="supply1" deviceset="GND" device=""/>
 <part name="GND13" library="supply1" deviceset="GND" device=""/>
@@
 <part name="SW-ACK" library="GW-devices" deviceset="SWITCH-TACTILE" device="-320.01E11WHT">
 <attribute name="MFGP" value="320.01E11WHT"/>
+<attribute name="PRICE" value="1.38"/>
 </part>
 <part name="U$3" library="GW-devices" deviceset="SWITCH-TACTILE" device="" value="SWITCH-TACTILE">
@@
 <attribute name="MFGN" value="Worldsemi"/>
 <attribute name="MFGP" value="WS2812"/>
+<attribute name="NOTES" value="DNP"/>
 </part>
 <part name="GND2" library="supply1" deviceset="GND" device=""/>
@@
 <instance part="+3V6" gate="G$1" x="-307.34" y="60.96"/>
 <instance part="GND5" gate="1" x="144.78" y="7.62"/>
-<instance part="SW-ACK" gate="G$1" x="124.46" y="27.94"/>
+<instance part="SW-ACK" gate="G$1" x="124.46" y="27.94">
+<attribute name="PRICE" x="124.46" y="27.94" size="1.778" layer="96" display="off"/>
+</instance>
 <instance part="U$3" gate="G$1" x="124.46" y="58.42">
 <attribute name="NOTES" x="124.46" y="58.42" size="1.778" layer="96" display="off"/>
@@
 <attribute name="MFGN" x="10.16" y="-66.04" size="1.778" layer="96" display="off"/>
 <attribute name="MFGP" x="10.16" y="-66.04" size="1.778" layer="96" display="off"/>
+<attribute name="NOTES" x="10.16" y="-66.04" size="1.778" layer="96" display="off"/>
 </instance>
 <instance part="GND2" gate="1" x="-7.62" y="-81.28"/>

Commit message: KW2 antenna, LasCon panel, PosCon fiducials
Added vertical MMCX connector to KW2 design & library; added panelized
version of LasCon (old and new design); added Adafruit library and
fiducials to new PosCon
Parts:
- added U$1, U$2, U$6, U$7, U$8, U$9: FIDUCIAL, adafruit:FIDUCIAL
Changed lines of the file:
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@@
 <layer number="54" name="bGND_GNDA" color="1" fill="9" visible="no" active="no"/>
 <layer number="56" name="wert" color="7" fill="1" visible="no" active="no"/>
+<layer number="57" name="tCAD" color="7" fill="1" visible="no" active="no"/>
 <layer number="91" name="Nets" color="2" fill="1" visible="yes" active="yes"/>
 <layer number="92" name="Busses" color="1" fill="1" visible="yes" active="yes"/>
@@
 <layer number="106" name="bPlate" color="14" fill="3" visible="yes" active="yes"/>
 <layer number="107" name="Crop" color="11" fill="1" visible="yes" active="yes"/>
+<layer number="108" name="fp8" color="7" fill="1" visible="no" active="yes"/>
+<layer number="109" name="fp9" color="7" fill="1" visible="no" active="yes"/>
+<layer number="110" name="fp0" color="7" fill="1" visible="no" active="yes"/>
+<layer number="111" name="LPC17xx" color="7" fill="1" visible="yes" active="yes"/>
+<layer number="112" name="tSilk" color="7" fill="1" visible="yes" active="yes"/>
 <layer number="116" name="Patch_BOT" color="9" fill="4" visible="yes" active="yes"/>
 <layer number="118" name="Rect_Pads" color="4" fill="1" visible="yes" active="yes"/>
 <layer number="121" name="_tsilk" color="7" fill="1" visible="yes" active="yes"/>
 <layer number="122" name="_bsilk" color="7" fill="1" visible="yes" active="yes"/>
+<layer number="123" name="tTestmark" color="7" fill="1" visible="no" active="yes"/>
+<layer number="124" name="bTestmark" color="7" fill="1" visible="no" active="yes"/>
 <layer number="125" name="_tNames" color="7" fill="1" visible="no" active="yes"/>
+<layer number="126" name="_bNames" color="7" fill="1" visible="yes" active="yes"/>
+<layer number="127" name="_tValues" color="7" fill="1" visible="yes" active="yes"/>
+<layer number="128" name="_bValues" color="7" fill="1" visible="yes" active="yes"/>
+<layer number="131" name="tAdjust" color="7" fill="1" visible="no" active="yes"/>
+<layer number="132" name="bAdjust" color="7" fill="1" visible="no" active="yes"/>
 <layer number="144" name="Drill_legend" color="7" fill="1" visible="no" active="yes"/>
+<layer number="150" name="Notes" color="7" fill="1" visible="no" active="yes"/>
 <layer number="151" name="HeatSink" color="7" fill="1" visible="yes" active="yes"/>
+<layer number="152" name="_bDocu" color="7" fill="1" visible="yes" active="yes"/>
+<layer number="153" name="FabDoc1" color="6" fill="1" visible="no" active="no"/>
+<layer number="154" name="FabDoc2" color="2" fill="1" visible="no" active="no"/>
+<layer number="155" name="FabDoc3" color="7" fill="15" visible="no" active="no"/>
+<layer number="199" name="Contour" color="7" fill="1" visible="yes" active="yes"/>
 <layer number="200" name="200bmp" color="1" fill="10" visible="yes" active="yes"/>
 <layer number="201" name="201bmp" color="2" fill="10" visible="yes" active="yes"/>
@@
 <layer number="223" name="223bmp" color="24" fill="1" visible="no" active="no"/>
 <layer number="224" name="224bmp" color="25" fill="1" visible="no" active="no"/>
+<layer number="248" name="Housing" color="7" fill="1" visible="yes" active="yes"/>
+<layer number="249" name="Edge" color="7" fill="1" visible="yes" active="yes"/>
 <layer number="250" name="Descript" color="3" fill="1" visible="no" active="no"/>
 <layer number="251" name="SMDround" color="12" fill="11" visible="no" active="no"/>
@@
 <part name="GND2" library="supply1" deviceset="GND" device=""/>
 <part name="+3V7" library="supply1" deviceset="+3V3" device=""/>
+<part name="U$1" library="adafruit" deviceset="FIDUCIAL" device=""/>
+<part name="U$2" library="adafruit" deviceset="FIDUCIAL" device=""/>
+<part name="U$6" library="adafruit" deviceset="FIDUCIAL" device=""/>
+<part name="U$7" library="adafruit" deviceset="FIDUCIAL" device=""/>
+<part name="U$8" library="adafruit" deviceset="FIDUCIAL" device=""/>
+<part name="U$9" library="adafruit" deviceset="FIDUCIAL" device=""/>
 </parts>
 <sheets>
@@
 <instance part="GND2" gate="1" x="-7.62" y="-81.28"/>
 <instance part="+3V7" gate="G$1" x="7.62" y="-43.18"/>
+<instance part="U$1" gate="G$1" x="-33.02" y="134.62"/>
+<instance part="U$2" gate="G$1" x="0" y="134.62"/>
+<instance part="U$6" gate="G$1" x="30.48" y="132.08"/>
+<instance part="U$7" gate="G$1" x="-25.4" y="109.22"/>
+<instance part="U$8" gate="G$1" x="5.08" y="104.14"/>
+<instance part="U$9" gate="G$1" x="33.02" y="104.14"/>
 </instances>
 <busses>

Commit message: PosCon parts, KW2 frontend, LasCon
Added part numbers for orange display, black buttons to PosCon. Worked
on frontend layout for KW2 and produced a new version of LasCon
Parts:
- J1-PROG, J2: MFGP 0955016649 -> 0955016889
- LED1, LED2: MFGN (none) -> Kingbright; MFGP (none) -> ACSA04-41SEKWA-F01; NOTES DNP -> (none)
- SW-ACK: PRICE 1.38 -> (none)
- U$3, U$4: MFGN (none) -> E-Switch; MFGP (none) -> TL3301PF160QG; NOTES DNP -> (none)
Changed lines of the file:
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@@
 <part name="+3V5" library="supply1" deviceset="+3V3" device=""/>
 <part name="LED2" library="GW-devices" deviceset="7SEGMENT-1DIGIT" device="SMD">
-<attribute name="NOTES" value="DNP"/>
+<attribute name="MFGN" value="Kingbright"/>
+<attribute name="MFGP" value="ACSA04-41SEKWA-F01 "/>
 </part>
 <part name="LED1" library="GW-devices" deviceset="7SEGMENT-1DIGIT" device="SMD">
-<attribute name="NOTES" value="DNP"/>
+<attribute name="MFGN" value="Kingbright"/>
+<attribute name="MFGP" value="ACSA04-41SEKWA-F01 "/>
 </part>
 <part name="+3V3" library="supply1" deviceset="+3V3" device=""/>
@@
 <part name="SW-ACK" library="GW-devices" deviceset="SWITCH-TACTILE" device="-320.01E11WHT">
 <attribute name="MFGP" value="320.01E11WHT"/>
-<attribute name="PRICE" value="1.38"/>
 </part>
 <part name="U$3" library="GW-devices" deviceset="SWITCH-TACTILE" device="" value="SWITCH-TACTILE">
-<attribute name="NOTES" value="DNP"/>
+<attribute name="MFGN" value="E-Switch"/>
+<attribute name="MFGP" value="TL3301PF160QG"/>
 </part>
 <part name="U$4" library="GW-devices" deviceset="SWITCH-TACTILE" device="" value="SWITCH-TACTILE">
-<attribute name="NOTES" value="DNP"/>
+<attribute name="MFGN" value="E-Switch"/>
+<attribute name="MFGP" value="TL3301PF160QG"/>
 </part>
 <part name="J1-PROG" library="GW-devices" deviceset="RJ45-8" device="">
 <attribute name="MFGN" value="Molex"/>
-<attribute name="MFGP" value="0955016649"/>
+<attribute name="MFGP" value="0955016889"/>
 <attribute name="PRICE" value="0.89"/>
 </part>
 <part name="J2" library="GW-devices" deviceset="RJ45-8" device="">
 <attribute name="MFGN" value="Molex"/>
-<attribute name="MFGP" value="0955016649"/>
+<attribute name="MFGP" value="0955016889"/>
 <attribute name="PRICE" value="0.89"/>
 </part>
@@
 <instance part="+3V5" gate="G$1" x="-73.66" y="81.28"/>
 <instance part="LED2" gate="G$1" x="-274.32" y="81.28">
-<attribute name="NOTES" x="-274.32" y="81.28" size="1.778" layer="96" display="off"/>
+<attribute name="MFGN" x="-274.32" y="81.28" size="1.778" layer="96" display="off"/>
+<attribute name="MFGP" x="-274.32" y="81.28" size="1.778" layer="96" display="off"/>
 </instance>
 <instance part="LED1" gate="G$1" x="-243.84" y="81.28">
-<attribute name="NOTES" x="-243.84" y="81.28" size="1.778" layer="96" display="off"/>
+<attribute name="MFGN" x="-243.84" y="81.28" size="1.778" layer="96" display="off"/>
+<attribute name="MFGP" x="-243.84" y="81.28" size="1.778" layer="96" display="off"/>
 </instance>
 <instance part="+3V3" gate="G$1" x="-307.34" y="109.22"/>
 <instance part="+3V6" gate="G$1" x="-307.34" y="60.96"/>
 <instance part="GND5" gate="1" x="144.78" y="7.62"/>
-<instance part="SW-ACK" gate="G$1" x="124.46" y="27.94">
-<attribute name="PRICE" x="124.46" y="27.94" size="1.778" layer="96" display="off"/>
-</instance>
+<instance part="SW-ACK" gate="G$1" x="124.46" y="27.94"/>
 <instance part="U$3" gate="G$1" x="124.46" y="58.42">
-<attribute name="NOTES" x="124.46" y="58.42" size="1.778" layer="96" display="off"/>
+<attribute name="MFGN" x="124.46" y="58.42" size="1.778" layer="96" display="off"/>
+<attribute name="MFGP" x="124.46" y="58.42" size="1.778" layer="96" display="off"/>
 </instance>
 <instance part="U$4" gate="G$1" x="124.46" y="43.18">
-<attribute name="NOTES" x="124.46" y="43.18" size="1.778" layer="96" display="off"/>
+<attribute name="MFGN" x="124.46" y="43.18" size="1.778" layer="96" display="off"/>
+<attribute name="MFGP" x="124.46" y="43.18" size="1.778" layer="96" display="off"/>
 </instance>
 <instance part="J1-PROG" gate="G$1" x="170.18" y="-20.32">
