File: LASCON.PCB/LasCon.sch (EAGLE design)
At the start: 17 parts

Commit message: Completed laser board
Finished routing, may need to redo flipped.
Connections:
- net +3V3: now also U$14.1, U$15.1, U$16.1
Other:
- moved on the sheet: U$5
Changed lines of the file:
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@@
 <part name="U$15" library="GW-devices" deviceset="RF-R" device="0805" value="24"/>
 <part name="U$16" library="GW-devices" deviceset="RF-R" device="0805" value="24"/>
+<part name="+3V5" library="supply1" deviceset="+3V3" device=""/>
 </parts>
 <sheets>
@@
 <instance part="U$2" gate="G$1" x="88.9" y="0" rot="R180"/>
 <instance part="U$3" gate="G$1" x="15.24" y="-20.32"/>
-<instance part="SUPPLY1" gate="GND" x="12.7" y="7.62"/>
-<instance part="SUPPLY2" gate="GND" x="-55.88" y="-15.24"/>
-<instance part="SUPPLY3" gate="GND" x="88.9" y="-15.24"/>
-<instance part="SUPPLY4" gate="GND" x="-7.62" y="-53.34"/>
+<instance part="SUPPLY1" gate="GND" x="12.7" y="5.08"/>
+<instance part="SUPPLY2" gate="GND" x="-55.88" y="-17.78"/>
+<instance part="SUPPLY3" gate="GND" x="88.9" y="-17.78"/>
+<instance part="SUPPLY4" gate="GND" x="-7.62" y="-55.88"/>
 <instance part="IC1" gate="G$1" x="12.7" y="17.78"/>
 <instance part="U$4" gate="G$1" x="-30.48" y="-35.56" rot="R90"/>
-<instance part="U$5" gate="G$1" x="-20.32" y="-35.56" rot="R90"/>
+<instance part="U$5" gate="G$1" x="-20.32" y="-33.02" rot="R90"/>
 <instance part="U$6" gate="G$1" x="66.04" y="-58.42" rot="R270"/>
 <instance part="U$7" gate="G$1" x="93.98" y="-58.42" rot="R270"/>
@@
 <instance part="U$15" gate="G$1" x="66.04" y="-121.92" rot="R90"/>
 <instance part="U$16" gate="G$1" x="71.12" y="-121.92" rot="R90"/>
+<instance part="+3V5" gate="G$1" x="50.8" y="-132.08"/>
 </instances>
 <busses>
@@
 <wire x1="88.9" y1="15.24" x2="78.74" y2="15.24" width="0.1524" layer="91"/>
 <wire x1="78.74" y1="15.24" x2="78.74" y2="10.16" width="0.1524" layer="91"/>
+<junction x="-15.24" y="17.78"/>
+<junction x="88.9" y="15.24"/>
+<junction x="-45.72" y="17.78"/>
 </segment>
 </net>
@@
 <pinref part="U$1" gate="G$1" pin="P$3"/>
 <wire x1="-66.04" y1="5.08" x2="-45.72" y2="5.08" width="0.1524" layer="91"/>
+<junction x="-45.72" y="5.08"/>
 </segment>
 </net>
@@
 <segment>
 <pinref part="U$1" gate="G$1" pin="P$6"/>
-<wire x1="-45.72" y1="0" x2="-43.18" y2="0" width="0.1524" layer="91"/>
-<wire x1="-43.18" y1="0" x2="-10.16" y2="0" width="0.1524" layer="91"/>
+<wire x1="-45.72" y1="0" x2="-10.16" y2="0" width="0.1524" layer="91"/>
 <wire x1="-10.16" y1="0" x2="-10.16" y2="-10.16" width="0.1524" layer="91"/>
 <pinref part="U$3" gate="G$1" pin="SDI"/>
 <wire x1="-10.16" y1="-10.16" x2="-2.54" y2="-10.16" width="0.1524" layer="91"/>
 <pinref part="U$1" gate="G$1" pin="P$5"/>
-<wire x1="-66.04" y1="0" x2="-43.18" y2="0" width="0.1524" layer="91"/>
+<wire x1="-66.04" y1="0" x2="-45.72" y2="0" width="0.1524" layer="91"/>
+<junction x="-45.72" y="0"/>
 </segment>
 </net>
@@
 <wire x1="78.74" y1="-5.08" x2="78.74" y2="-12.7" width="0.1524" layer="91"/>
 <wire x1="78.74" y1="-12.7" x2="88.9" y2="-12.7" width="0.1524" layer="91"/>
+<wire x1="88.9" y1="-12.7" x2="88.9" y2="-15.24" width="0.1524" layer="91"/>
+<wire x1="88.9" y1="-15.24" x2="88.9" y2="-12.7" width="0.1524" layer="91"/>
 <wire x1="88.9" y1="-12.7" x2="99.06" y2="-12.7" width="0.1524" layer="91"/>
 <pinref part="SUPPLY3" gate="GND" pin="GND"/>
+<junction x="88.9" y="-12.7"/>
+<junction x="88.9" y="-15.24"/>
 </segment>
 <segment>
@@
 <wire x1="-7.62" y1="-35.56" x2="-7.62" y2="-50.8" width="0.1524" layer="91"/>
 <pinref part="U$4" gate="G$1" pin="1"/>
-<wire x1="-30.48" y1="-40.64" x2="-25.4" y2="-40.64" width="0.1524" layer="91"/>
+<wire x1="-7.62" y1="-50.8" x2="-7.62" y2="-53.34" width="0.1524" layer="91"/>
+<wire x1="-30.48" y1="-40.64" x2="-30.48" y2="-43.18" width="0.1524" layer="91"/>
 <pinref part="U$5" gate="G$1" pin="1"/>
-<wire x1="-25.4" y1="-40.64" x2="-22.86" y2="-40.64" width="0.1524" layer="91"/>
-<wire x1="-22.86" y1="-40.64" x2="-20.32" y2="-40.64" width="0.1524" layer="91"/>
+<wire x1="-30.48" y1="-43.18" x2="-22.86" y2="-43.18" width="0.1524" layer="91"/>
+<wire x1="-22.86" y1="-43.18" x2="-20.32" y2="-43.18" width="0.1524" layer="91"/>
+<wire x1="-7.62" y1="-53.34" x2="-7.62" y2="-50.8" width="0.1524" layer="91"/>
 <wire x1="-7.62" y1="-50.8" x2="-22.86" y2="-50.8" width="0.1524" layer="91"/>
-<wire x1="-22.86" y1="-50.8" x2="-22.86" y2="-40.64" width="0.1524" layer="91"/>
+<wire x1="-22.86" y1="-50.8" x2="-22.86" y2="-43.18" width="0.1524" layer="91"/>
 <pinref part="U$12" gate="G$1" pin="1"/>
-<wire x1="-20.32" y1="-40.64" x2="-12.7" y2="-40.64" width="0.1524" layer="91"/>
+<wire x1="-20.32" y1="-38.1" x2="-20.32" y2="-43.18" width="0.1524" layer="91"/>
+<wire x1="-20.32" y1="-43.18" x2="-12.7" y2="-43.18" width="0.1524" layer="91"/>
+<wire x1="-12.7" y1="-43.18" x2="-12.7" y2="-40.64" width="0.1524" layer="91"/>
+<junction x="-22.86" y="-43.18"/>
+<junction x="-20.32" y="-43.18"/>
+<junction x="-7.62" y="-50.8"/>
+<junction x="-7.62" y="-53.34"/>
 </segment>
 <segment>
 <pinref part="SUPPLY1" gate="GND" pin="GND"/>
 <pinref part="IC1" gate="G$1" pin="GND"/>
-<wire x1="12.7" y1="10.16" x2="12.7" y2="12.7" width="0.1524" layer="91"/>
+<wire x1="12.7" y1="7.62" x2="12.7" y2="12.7" width="0.1524" layer="91"/>
 <pinref part="IC1" gate="G$1" pin="P$1"/>
-<wire x1="12.7" y1="10.16" x2="17.78" y2="10.16" width="0.1524" layer="91"/>
-<wire x1="17.78" y1="10.16" x2="20.32" y2="10.16" width="0.1524" layer="91"/>
-<wire x1="20.32" y1="10.16" x2="20.32" y2="12.7" width="0.1524" layer="91"/>
+<wire x1="12.7" y1="7.62" x2="20.32" y2="7.62" width="0.1524" layer="91"/>
+<wire x1="20.32" y1="7.62" x2="20.32" y2="12.7" width="0.1524" layer="91"/>
 <pinref part="U$10" gate="G$1" pin="2"/>
-<wire x1="17.78" y1="10.16" x2="20.32" y2="10.16" width="0.1524" layer="91"/>
-<wire x1="20.32" y1="10.16" x2="20.32" y2="5.08" width="0.1524" layer="91"/>
+<junction x="20.32" y="7.62"/>
+<junction x="12.7" y="7.62"/>
+<wire x1="20.32" y1="7.62" x2="20.32" y2="5.08" width="0.1524" layer="91"/>
 </segment>
 <segment>
 <pinref part="SUPPLY2" gate="GND" pin="GND"/>
 <pinref part="U$1" gate="G$1" pin="P$7"/>
+<wire x1="-55.88" y1="-15.24" x2="-55.88" y2="-12.7" width="0.1524" layer="91"/>
 <wire x1="-55.88" y1="-12.7" x2="-66.04" y2="-12.7" width="0.1524" layer="91"/>
 <wire x1="-66.04" y1="-12.7" x2="-66.04" y2="-5.08" width="0.1524" layer="91"/>
 <pinref part="U$1" gate="G$1" pin="P$8"/>
+<wire x1="-55.88" y1="-15.24" x2="-55.88" y2="-12.7" width="0.1524" layer="91"/>
 <wire x1="-55.88" y1="-12.7" x2="-45.72" y2="-12.7" width="0.1524" layer="91"/>
 <wire x1="-45.72" y1="-12.7" x2="-45.72" y2="-5.08" width="0.1524" layer="91"/>
+<junction x="-55.88" y="-12.7"/>
+<junction x="-55.88" y="-15.24"/>
 </segment>
 </net>
@@
 <pinref part="U$2" gate="G$1" pin="P$5"/>
 <wire x1="99.06" y1="5.08" x2="78.74" y2="5.08" width="0.1524" layer="91"/>
+<junction x="78.74" y="5.08"/>
 </segment>
 </net>
@@
 <pinref part="U$2" gate="G$1" pin="P$3"/>
 <wire x1="99.06" y1="0" x2="78.74" y2="0" width="0.1524" layer="91"/>
+<junction x="78.74" y="0"/>
 </segment>
 </net>
@@
 <pinref part="U$5" gate="G$1" pin="2"/>
 <wire x1="-2.54" y1="-25.4" x2="-20.32" y2="-25.4" width="0.1524" layer="91"/>
-<wire x1="-20.32" y1="-25.4" x2="-20.32" y2="-30.48" width="0.1524" layer="91"/>
+<wire x1="-20.32" y1="-25.4" x2="-20.32" y2="-27.94" width="0.1524" layer="91"/>
 </segment>
 </net>
@@
 <wire x1="76.2" y1="-81.28" x2="66.04" y2="-81.28" width="0.1524" layer="91"/>
 <wire x1="66.04" y1="-81.28" x2="66.04" y2="-83.82" width="0.1524" layer="91"/>
+<junction x="93.98" y="-43.18"/>
 </segment>
 </net>
@@
 <pinref part="U$10" gate="G$1" pin="1"/>
 <wire x1="27.94" y1="5.08" x2="30.48" y2="5.08" width="0.1524" layer="91"/>
+<junction x="30.48" y="7.62"/>
+<junction x="30.48" y="5.08"/>
 </segment>
 <segment>
@@
 <pinref part="U$11" gate="G$1" pin="PWR"/>
 <wire x1="45.72" y1="-35.56" x2="45.72" y2="-50.8" width="0.1524" layer="91"/>
+</segment>
+<segment>
+<pinref part="U$14" gate="G$1" pin="1"/>
+<wire x1="60.96" y1="-127" x2="60.96" y2="-134.62" width="0.1524" layer="91"/>
+<pinref part="+3V5" gate="G$1" pin="+3V3"/>
+<wire x1="60.96" y1="-134.62" x2="50.8" y2="-134.62" width="0.1524" layer="91"/>
+<pinref part="U$15" gate="G$1" pin="1"/>
+<wire x1="66.04" y1="-127" x2="66.04" y2="-134.62" width="0.1524" layer="91"/>
+<wire x1="66.04" y1="-134.62" x2="60.96" y2="-134.62" width="0.1524" layer="91"/>
+<pinref part="U$16" gate="G$1" pin="1"/>
+<wire x1="71.12" y1="-127" x2="71.12" y2="-134.62" width="0.1524" layer="91"/>
+<wire x1="71.12" y1="-134.62" x2="66.04" y2="-134.62" width="0.1524" layer="91"/>
+<junction x="60.96" y="-134.62"/>
+<junction x="66.04" y="-134.62"/>
+<junction x="71.12" y="-134.62"/>
 </segment>
 </net>
@@
 <wire x1="55.88" y1="-81.28" x2="60.96" y2="-81.28" width="0.1524" layer="91"/>
 <wire x1="60.96" y1="-81.28" x2="60.96" y2="-83.82" width="0.1524" layer="91"/>
+<junction x="66.04" y="-43.18"/>
 </segment>
 </net>
@@
 <wire x1="27.94" y1="-76.2" x2="71.12" y2="-76.2" width="0.1524" layer="91"/>
 <wire x1="71.12" y1="-76.2" x2="71.12" y2="-83.82" width="0.1524" layer="91"/>
+<junction x="40.64" y="-40.64"/>
 </segment>
 </net>
@@
 </sheet>
 </sheets>
+<errors>
+</errors>
 </schematic>
 </drawing>

Commit message: LasCon BOM
Updated LasCon parts
Parts:
- IC1: MPN (none) -> MCP1804T-3302I/DB
- U$8, U$9: MFGN (none) -> Keystone Electronics; MFGP (none) -> 7774
Changed lines of the file:
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@@
 <part name="SUPPLY3" library="supply2" deviceset="GND" device=""/>
 <part name="SUPPLY4" library="supply2" deviceset="GND" device=""/>
-<part name="IC1" library="microchip" deviceset="MCP1804T-3302I" device=""/>
+<part name="IC1" library="microchip" deviceset="MCP1804T-3302I" device="">
+<attribute name="MPN" value="MCP1804T-3302I/DB"/>
+</part>
 <part name="U$4" library="GW-devices" deviceset="RF-R" device="0805" value="24"/>
 <part name="U$5" library="GW-devices" deviceset="RF-R" device="0805" value="24"/>
@@
 <part name="+3V2" library="supply1" deviceset="+3V3" device=""/>
 <part name="+3V3" library="supply1" deviceset="+3V3" device=""/>
-<part name="U$8" library="GW-devices" deviceset="90DEGMNT" device=""/>
-<part name="U$9" library="GW-devices" deviceset="90DEGMNT" device=""/>
+<part name="U$8" library="GW-devices" deviceset="90DEGMNT" device="">
+<attribute name="MFGN" value="Keystone Electronics"/>
+<attribute name="MFGP" value="7774"/>
+</part>
+<part name="U$9" library="GW-devices" deviceset="90DEGMNT" device="">
+<attribute name="MFGN" value="Keystone Electronics"/>
+<attribute name="MFGP" value="7774"/>
+</part>
 <part name="U$10" library="GW-devices" deviceset="RF-C" device="0805"/>
 <part name="U$11" library="GW-devices" deviceset="LASER" device=""/>
@@
 <instance part="+3V2" gate="G$1" x="71.12" y="-33.02"/>
 <instance part="+3V3" gate="G$1" x="99.06" y="-30.48"/>
-<instance part="U$8" gate="G$1" x="-60.96" y="-53.34"/>
-<instance part="U$9" gate="G$1" x="119.38" y="-53.34"/>
+<instance part="U$8" gate="G$1" x="-60.96" y="-53.34">
+<attribute name="MFGN" x="-60.96" y="-53.34" size="1.778" layer="96" display="off"/>
+<attribute name="MFGP" x="-60.96" y="-53.34" size="1.778" layer="96" display="off"/>
+</instance>
+<instance part="U$9" gate="G$1" x="119.38" y="-53.34">
+<attribute name="MFGN" x="119.38" y="-53.34" size="1.778" layer="96" display="off"/>
+<attribute name="MFGP" x="119.38" y="-53.34" size="1.778" layer="96" display="off"/>
+</instance>
 <instance part="U$10" gate="G$1" x="25.4" y="5.08" rot="R270"/>
 <instance part="U$11" gate="G$1" x="40.64" y="-58.42" rot="R270"/>
